Commit message: Update robot descriptions and launch files for Webots integration

File: rc_manipulators_description/urdf/arm/universal_robots.urdf.xacro (robot description, xacro)
@@ -2,5 +2,6 @@
 <robot xmlns:xacro="http://ros.org/wiki/xacro">
   <xacro:arg name="is_sim" default="false"/>
-  <xacro:arg name="use_mock_hardware" default="false"/>
+  <xacro:arg name="use_fake_hardware" default="false"/>
+  <xacro:arg name="use_mock_hardware" default="$(arg use_fake_hardware)"/>
   <xacro:arg name="use_manipulation_controllers" default="false"/>
   <xacro:include filename="$(find ur_description)/urdf/ur_macro.xacro"/>
@@ -87,5 +88,5 @@
     </xacro:if>
     <!-- Default Simulation Parameters -->
-    <xacro:property name="_use_mock_hardware" value="false" />
+    <xacro:property name="_use_mock_hardware" value="$(arg use_mock_hardware)" />
     <xacro:property name="_mock_sensor_commands" value="false" />
     <xacro:property name="_sim_gazebo" value="false" />
@@ -223,5 +224,6 @@
       <ros2_control name="${name}_hardware" type="system">
         <hardware>
-          <plugin>gz_ros2_control/GazeboSimSystem</plugin>
+          <!-- <plugin>gz_ros2_control/GazeboSimSystem</plugin> -->
+          <plugin>webots_ros2_control::Ros2ControlSystem</plugin>
         </hardware>
         <joint name="${name}_shoulder_pan_joint">
@@ -256,8 +258,8 @@
         </joint>
       </ros2_control>
-      <gazebo>
-        <plugin filename="gz_ros2_control-system"
-                name="gz_ros2_control::GazeboSimROS2ControlPlugin"/>
-      </gazebo>
+      <!-- <gazebo> -->
+        <!-- <plugin filename="gz_ros2_control-system" -->
+                <!-- name="gz_ros2_control::GazeboSimROS2ControlPlugin"/> -->
+      <!-- </gazebo> -->
     </xacro:if>
     <!-- REAL ROBOT: only include the UR driver when NOT sim -->

File: rc_manipulators_description/urdf/gripper/robotiq_2f_140.urdf.xacro (robot description, xacro)
@@ -294,5 +294,6 @@
           </xacro:if>
           <xacro:if value="${sim_gazebo}">
-            <plugin>gz_ros2_control/GazeboSimSystem</plugin>
+            <!-- <plugin>gz_ros2_control/GazeboSimSystem</plugin> -->
+            <plugin>webots_ros2_control::Ros2ControlSystem</plugin>
           </xacro:if>
           <xacro:if value="${use_fake_hardware}">

File: rc_platform_description/urdf/a300/a300.urdf.xacro (robot description, xacro)
@@ -17,19 +17,7 @@
     <xacro:property name="wheel_track" value="0.562"/>
     <!-- Chassis Positions relative to center of rotation -->
-    <xacro:if value="${control == 'diff_4wd' or control == 'omni_4wd'}">
-      <xacro:property name="chassis_x" value="0"/>
-      <xacro:property name="chassis_y" value="0"/>
-      <xacro:property name="chassis_z" value="0"/>
-    </xacro:if>
-    <xacro:if value="${control == 'diff_fwd'}">
-      <xacro:property name="chassis_x" value="${-wheel_base / 2}"/>
-      <xacro:property name="chassis_y" value="0"/>
-      <xacro:property name="chassis_z" value="0"/>
-    </xacro:if>
-    <xacro:if value="${control == 'diff_rwd'}">
-      <xacro:property name="chassis_x" value="${wheel_base / 2}"/>
-      <xacro:property name="chassis_y" value="0"/>
-      <xacro:property name="chassis_z" value="0"/>
-    </xacro:if>
+    <xacro:property name="chassis_x" value="0"/>
+    <xacro:property name="chassis_y" value="0"/>
+    <xacro:property name="chassis_z" value="0"/>
     <!-- Suspension Beam Mounting Positions -->
     <xacro:property name="chassis_suspension_mount_x" value="0.0"/>
@@ -127,5 +115,5 @@
     <!-- Hardware  -->
     <xacro:if value="$(arg is_sim)">
-      <xacro:property name="hardware_plugin" value="gz_ros2_control/GazeboSimSystem"/>
+      <xacro:property name="hardware_plugin" value="webots_ros2_control::Ros2ControlSystem"/>
     </xacro:if>
     <xacro:unless value="$(arg is_sim)">
@@ -143,18 +131,9 @@
     <!-- Base Footprint: on the ground below the robot -->
     <link name="base_footprint"/>
-    <xacro:if value="${control == 'diff_4wd' or control == 'omni_4wd' or control == 'diff_fwd'}">
-      <joint name="base_footprint_joint" type="fixed">
-        <origin xyz="0 0 ${front_wheel_radius}" rpy="0 0 0" />
-        <parent link="chassis_link" />
-        <child link="base_footprint" />
-      </joint>
-    </xacro:if>
-    <xacro:if value="${control == 'diff_rwd'}">
-      <joint name="base_footprint_joint" type="fixed">
-        <origin xyz="0 0 ${rear_wheel_radius}" rpy="0 0 0" />
-        <parent link="chassis_link" />
-        <child link="base_footprint" />
-      </joint>
-    </xacro:if>
+    <joint name="base_footprint_joint" type="fixed">
+      <origin xyz="0 0 ${front_wheel_radius}" rpy="0 0 0" />
+      <parent link="chassis_link" />
+      <child link="base_footprint" />
+    </joint>
   </xacro:macro>
 </robot>

File: rc_platform_description/urdf/a300/drivetrain/wheels.urdf.xacro (robot description, xacro)
@@ -3,70 +3,23 @@
   <xacro:macro name="a300_drivetrain_wheels" params="front_wheels rear_wheels">
     <xacro:include filename="$(find rc_platform_description)/urdf/a300/drivetrain/wheels/outdoor.urdf.xacro" />
-    <xacro:include filename="$(find rc_platform_description)/urdf/a300/drivetrain/wheels/mecanum.urdf.xacro" />
-    <xacro:include filename="$(find rc_platform_description)/urdf/a300/drivetrain/wheels/caster.urdf.xacro" />
     <xacro:include filename="$(find rc_platform_description)/urdf/a300/drivetrain/motor.urdf.xacro" />
-    <xacro:include filename="$(find rc_platform_description)/urdf/a300/drivetrain/caster_flange.urdf.xacro" />
-    <!-- Front Wheels -->
-    <xacro:if value="${front_wheels == 'outdoor'}">
-      <xacro:property name="front_wheel_radius" value="${a300_outdoor_wheel_radius}" scope="parent"/>
-      <xacro:property name="front_wheel_width" value="${a300_outdoor_wheel_width}" scope="parent"/>
-      <!-- Motors -->
-      <xacro:a300_motor prefix="front" side="left"/>
-      <xacro:a300_motor prefix="front" side="right"/>
-      <!-- Wheels -->
-      <xacro:a300_outdoor_wheel prefix="front" side="left"/>
-      <xacro:a300_outdoor_wheel prefix="front" side="right"/>
-    </xacro:if>
-    <xacro:if value="${front_wheels == 'mecanum'}">
-      <xacro:property name="front_wheel_radius" value="${a300_mecanum_wheel_radius}" scope="parent"/>
-      <xacro:property name="front_wheel_width" value="${a300_mecanum_wheel_width}" scope="parent"/>
-      <!-- Motors -->
-      <xacro:a300_motor prefix="front" side="left"/>
-      <xacro:a300_motor prefix="front" side="right"/>
-      <!-- Wheels -->
-      <xacro:a300_mecanum_wheel prefix="front" side="left"/>
-      <xacro:a300_mecanum_wheel prefix="front" side="right"/>
-    </xacro:if>
-    <xacro:if value="${front_wheels == 'caster'}">
-      <xacro:property name="front_wheel_radius" value="${a300_caster_wheel_radius}" scope="parent"/>
-      <xacro:property name="front_wheel_width" value="${a300_caster_wheel_width}" scope="parent"/>
-      <!-- Flanges -->
-      <xacro:a300_caster_flange prefix="front" side="left"/>
-      <xacro:a300_caster_flange prefix="front" side="right"/>
-      <!-- Wheels -->
-      <xacro:a300_caster_wheel prefix="front" side="left"/>
-      <xacro:a300_caster_wheel prefix="front" side="right"/>
-    </xacro:if>
-    <!-- Rear Wheels -->
-    <xacro:if value="${rear_wheels == 'outdoor'}">
-      <xacro:property name="rear_wheel_radius" value="${a300_outdoor_wheel_radius}" scope="parent"/>
-      <xacro:property name="rear_wheel_width" value="${a300_outdoor_wheel_width}" scope="parent"/>
-      <!-- Motors -->
-      <xacro:a300_motor prefix="rear" side="left"/>
-      <xacro:a300_motor prefix="rear" side="right"/>
-      <!-- Wheels -->
-      <xacro:a300_outdoor_wheel prefix="rear" side="left"/>
-      <xacro:a300_outdoor_wheel prefix="rear" side="right"/>
-    </xacro:if>
-    <xacro:if value="${rear_wheels == 'mecanum'}">
-      <xacro:property name="rear_wheel_radius" value="${a300_mecanum_wheel_radius}" scope="parent"/>
-      <xacro:property name="rear_wheel_width" value="${a300_mecanum_wheel_width}" scope="parent"/>
-      <!-- Motors -->
-      <xacro:a300_motor prefix="rear" side="left"/>
-      <xacro:a300_motor prefix="rear" side="right"/>
-      <!-- Wheels -->
-      <xacro:a300_mecanum_wheel prefix="rear" side="left"/>
-      <xacro:a300_mecanum_wheel prefix="rear" side="right"/>
-    </xacro:if>
-    <xacro:if value="${rear_wheels == 'caster'}">
-      <xacro:property name="rear_wheel_radius" value="${a300_caster_wheel_radius}" scope="parent"/>
-      <xacro:property name="rear_wheel_width" value="${a300_caster_wheel_width}" scope="parent"/>
-      <!-- Flanges -->
-      <xacro:a300_caster_flange prefix="rear" side="left"/>
-      <xacro:a300_caster_flange prefix="rear" side="right"/>
-      <!-- Wheels -->
-      <xacro:a300_caster_wheel prefix="rear" side="left"/>
-      <xacro:a300_caster_wheel prefix="rear" side="right"/>
-    </xacro:if>
+    <!-- Front Wheels (Outdoor Only) -->
+    <xacro:property name="front_wheel_radius" value="${a300_outdoor_wheel_radius}" scope="parent"/>
+    <xacro:property name="front_wheel_width" value="${a300_outdoor_wheel_width}" scope="parent"/>
+    <!-- Motors -->
+    <xacro:a300_motor prefix="front" side="left"/>
+    <xacro:a300_motor prefix="front" side="right"/>
+    <!-- Wheels -->
+    <xacro:a300_outdoor_wheel prefix="front" side="left"/>
+    <xacro:a300_outdoor_wheel prefix="front" side="right"/>
+    <!-- Rear Wheels (Outdoor Only) -->
+    <xacro:property name="rear_wheel_radius" value="${a300_outdoor_wheel_radius}" scope="parent"/>
+    <xacro:property name="rear_wheel_width" value="${a300_outdoor_wheel_width}" scope="parent"/>
+    <!-- Motors -->
+    <xacro:a300_motor prefix="rear" side="left"/>
+    <xacro:a300_motor prefix="rear" side="right"/>
+    <!-- Wheels -->
+    <xacro:a300_outdoor_wheel prefix="rear" side="left"/>
+    <xacro:a300_outdoor_wheel prefix="rear" side="right"/>
   </xacro:macro>
 </robot>

File: rc_platform_description/urdf/a300/drivetrain/wheels/outdoor.urdf.xacro (robot description, xacro)
@@ -28,14 +28,14 @@
       </collision>
     </link>
-    <gazebo>
-      <plugin filename="libgz-sim-wheel-slip-system.so" name="gz::sim::systems::WheelSlip">
-        <wheel link_name="${prefix}_${side}_wheel_link">
-          <slip_compliance_lateral>0.75</slip_compliance_lateral>
-          <slip_compliance_longitudinal>0.75</slip_compliance_longitudinal>
-          <wheel_normal_force>113</wheel_normal_force>
-          <wheel_radius>${a300_outdoor_wheel_radius}</wheel_radius>
-        </wheel>
-      </plugin>
-    </gazebo>
+    <!-- <gazebo> -->
+      <!-- <plugin filename="libgz-sim-wheel-slip-system.so" name="gz::sim::systems::WheelSlip"> -->
+        <!-- <wheel link_name="${prefix}_${side}_wheel_link"> -->
+          <!-- <slip_compliance_lateral>0.75</slip_compliance_lateral> -->
+          <!-- <slip_compliance_longitudinal>0.75</slip_compliance_longitudinal> -->
+          <!-- <wheel_normal_force>113</wheel_normal_force> -->
+          <!-- <wheel_radius>${a300_outdoor_wheel_radius}</wheel_radius> -->
+        <!-- </wheel> -->
+      <!-- </plugin> -->
+    <!-- </gazebo> -->
     <joint name="${prefix}_${side}_wheel_joint" type="continuous">
       <parent link="${prefix}_${side}_motor_mount"/>

File: rc_platform_description/urdf/generic/drivetrain/control/diff_4wd.urdf.xacro (robot description, xacro)
@@ -2,7 +2,32 @@
 <robot xmlns:xacro="http://ros.org/wiki/xacro" xmlns:gz="http://gazebosim.org/schema" name="generic_drivetrain_control_diff_4wd">
   <xacro:macro name="generic_drivetrain_control_diff_4wd" params="name hardware_plugin">
-    <!-- This is the same as omni_4wd -->
-    <xacro:include filename="$(find rc_platform_description)/urdf/generic/drivetrain/control/omni_4wd.urdf.xacro"/>
-    <xacro:generic_drivetrain_control_omni_4wd name="${name}" hardware_plugin="${hardware_plugin}"/>
+    <!-- Gazebo Controller -->
+    <xacro:include filename="$(find rc_platform_description)/urdf/generic/gazebo.urdf.xacro"/>
+    <!-- ROS2 controls -->
+    <ros2_control name="${name}_hardware" type="system">
+      <hardware>
+        <plugin>${hardware_plugin}</plugin>
+      </hardware>
+      <joint name="front_left_wheel_joint">
+        <command_interface name="velocity"/>
+        <state_interface name="position"/>
+        <state_interface name="velocity"/>
+      </joint>
+      <joint name="front_right_wheel_joint">
+        <command_interface name="velocity"/>
+        <state_interface name="position"/>
+        <state_interface name="velocity"/>
+      </joint>
+      <joint name="rear_left_wheel_joint">
+        <command_interface name="velocity"/>
+        <state_interface name="position"/>
+        <state_interface name="velocity"/>
+      </joint>
+      <joint name="rear_right_wheel_joint">
+        <command_interface name="velocity"/>
+        <state_interface name="position"/>
+        <state_interface name="velocity"/>
+      </joint>
+    </ros2_control>
   </xacro:macro>
 </robot>

File: rc_platform_description/urdf/generic/drivetrain/drivetrain.urdf.xacro (robot description, xacro)
@@ -2,24 +2,7 @@
 <robot xmlns:xacro="http://ros.org/wiki/xacro" xmlns:gz="http://gazebosim.org/schema" name="generic_drivetrain">
   <xacro:macro name="generic_drivetrain" params="name control front_wheels rear_wheels hardware_plugin">
-    <!-- Omni drivetrain -->
-    <xacro:if value="${control == 'omni_4wd'}">
-      <xacro:include filename="$(find rc_platform_description)/urdf/generic/drivetrain/control/omni_4wd.urdf.xacro"/>
-      <xacro:generic_drivetrain_control_omni_4wd name="${name}" hardware_plugin="${hardware_plugin}"/>
-    </xacro:if>
     <!-- Diff 4WD drivetrain -->
-    <xacro:if value="${control == 'diff_4wd'}">
-      <xacro:include filename="$(find rc_platform_description)/urdf/generic/drivetrain/control/diff_4wd.urdf.xacro"/>
-      <xacro:generic_drivetrain_control_diff_4wd name="${name}" hardware_plugin="${hardware_plugin}"/>
-    </xacro:if>
-    <!-- Diff FWD drivetrain -->
-    <xacro:if value="${control == 'diff_fwd'}">
-      <xacro:include filename="$(find rc_platform_description)/urdf/generic/drivetrain/control/diff_fwd.urdf.xacro"/>
-      <xacro:generic_drivetrain_control_diff_fwd name="${name}" hardware_plugin="${hardware_plugin}"/>
-    </xacro:if>
-    <!-- Diff RWD drivetrain -->
-    <xacro:if value="${control == 'diff_rwd'}">
-      <xacro:include filename="$(find rc_platform_description)/urdf/generic/drivetrain/control/diff_rwd.urdf.xacro"/>
-      <xacro:generic_drivetrain_control_diff_rwd name="${name}" hardware_plugin="${hardware_plugin}"/>
-    </xacro:if>
+    <xacro:include filename="$(find rc_platform_description)/urdf/generic/drivetrain/control/diff_4wd.urdf.xacro"/>
+    <xacro:generic_drivetrain_control_diff_4wd name="${name}" hardware_plugin="${hardware_plugin}"/>
   </xacro:macro>
 </robot>

File: rc_platform_description/urdf/generic/gazebo.urdf.xacro (robot description, xacro)
@@ -2,22 +2,10 @@
 <robot xmlns:xacro="http://ros.org/wiki/xacro">
   <xacro:if value="$(arg is_sim)">
-    <gazebo>
-      <plugin filename="libgz_ros2_control-system.so" name="gz_ros2_control::GazeboSimROS2ControlPlugin">
-        <parameters>$(arg gazebo_controllers)</parameters>
-        <ros>
-          <remapping>~/odom:=platform/odom</remapping>
-          <remapping>~/cmd_vel:=platform/cmd_vel</remapping>
-          <remapping>/tf:=tf</remapping>
-          <remapping>/tf_static:=tf_static</remapping>
-          <remapping>/diagnostics:=diagnostics</remapping>
-          <remapping>/dynamic_joint_states:=platform/dynamic_joint_states</remapping>
-          <remapping>joint_states:=platform/joint_states</remapping>
-          <remapping>~/reference:=platform/cmd_vel</remapping>
-          <remapping>~/odometry:=platform/odom</remapping>
-          <namespace>$(arg namespace)</namespace>
-        </ros>
-      </plugin>
-    </gazebo>
-    <gazebo>
+    <ros2_control name="WebotsControl" type="system">
+      <hardware>
+        <plugin>webots_ros2_control::Ros2ControlSystem</plugin>
+      </hardware>
+    </ros2_control>
+    <!-- <gazebo>
       <plugin filename="libgz-sim-pose-publisher-system.so" name="gz::sim::systems::PosePublisher">
         <publish_link_pose>true</publish_link_pose>
@@ -26,5 +14,5 @@
         <update_frequency>50</update_frequency>
       </plugin>
-    </gazebo>
+    </gazebo> -->
   </xacro:if>
 </robot>
