Commit message: + Robot and spawned correctly + Ros2 controllers are configured

File: rc_common/robot.urdf.xacro (robot description, xacro)
@@ -24,10 +24,10 @@
   <!-- lidar2d_0 -->
   <xacro:include filename="$(find rc_sensors_description)/urdf/hokuyo_ust.urdf.xacro"/>
-  <xacro:hokuyo_ust name="lidar2d_0" parent_link="top_plate_front_mount" ang_res="0.5" min_ang="-3.141592653589793" max_ang="3.141592653589793" min_range="0.05" max_range="25.0" update_rate="40">
+  <xacro:hokuyo_ust name="lidar2d_0" parent_link="top_plate_link" ang_res="0.5" min_ang="-3.141592653589793" max_ang="3.141592653589793" min_range="0.05" max_range="25.0" update_rate="40">
     <origin xyz="-0.1 0.0 0.0" rpy="0.0 0.0 0.0"/>
   </xacro:hokuyo_ust>
   <!-- lidar2d_1 -->
   <xacro:include filename="$(find rc_sensors_description)/urdf/hokuyo_ust.urdf.xacro"/>
-  <xacro:hokuyo_ust name="lidar2d_1" parent_link="top_plate_rear_mount" ang_res="0.5" min_ang="-3.141592653589793" max_ang="3.141592653589793" min_range="0.05" max_range="25.0" update_rate="40">
+  <xacro:hokuyo_ust name="lidar2d_1" parent_link="top_plate_link" ang_res="0.5" min_ang="-3.141592653589793" max_ang="3.141592653589793" min_range="0.05" max_range="25.0" update_rate="40">
     <origin xyz="0.1 0.0 0.0" rpy="0.0 0.0 3.1415"/>
   </xacro:hokuyo_ust>
@@ -45,10 +45,10 @@
   <!-- arm_0 -->
   <xacro:include filename="$(find rc_manipulators_description)/urdf/arm/universal_robots.urdf.xacro"/>
-  <xacro:universal_robots name="arm_0" parent_link="default_mount" ur_type="ur5e" kinematics_parameters_file="$(find ur_description)/config/ur5e/default_kinematics.yaml" headless_mode="False" robot_ip="192.168.131.40">
+  <xacro:universal_robots name="arm_0" parent_link="top_plate_link" ur_type="ur5e" kinematics_parameters_file="$(find rc_manipulators_description)/urdf/arm/ur_description_webots/config/ur5e/default_kinematics.yaml" headless_mode="False" robot_ip="192.168.131.40">
     <origin xyz="0.0 0.0 0.0" rpy="0.0 0.0 0.0"/>
   </xacro:universal_robots>
   <!-- arm_0_gripper -->
   <xacro:include filename="$(find rc_manipulators_description)/urdf/gripper/robotiq_2f_140.urdf.xacro"/>
-  <xacro:robotiq_2f_140 name="arm_0_gripper" parent_link="arm_0_tool0">
+  <xacro:robotiq_2f_140 name="arm_0_gripper" parent_link="arm_0_tool0" use_controllers="true" sim_gazebo="true">
     <origin xyz="0.0 0.0 0.0" rpy="0.0 0.0 0.0"/>
   </xacro:robotiq_2f_140>

File: rc_manipulators_description/urdf/arm/universal_robots.urdf.xacro (robot description, xacro)
@@ -5,5 +5,5 @@
   <xacro:arg name="use_mock_hardware" default="$(arg use_fake_hardware)"/>
   <xacro:arg name="use_manipulation_controllers" default="false"/>
-  <xacro:include filename="$(find ur_description)/urdf/ur_macro.xacro"/>
+  <xacro:include filename="$(find rc_manipulators_description)/urdf/arm/ur_description_webots/urdf/ur_macro.xacro"/>
   <xacro:macro name="universal_robots" params="
     name
@@ -51,8 +51,8 @@
     <xacro:property name="_tf_prefix" value="${name}_" lazy_eval="false"/>
     <xacro:property name="_initial_positions" value="${dict(shoulder_pan_joint=0.0,shoulder_lift_joint=-1.57,elbow_joint=0.0,wrist_1_joint=-1.57,wrist_2_joint=0.0,wrist_3_joint=0.0)}" lazy_eval="false"/>
-    <xacro:property name="_joint_limits_parameters_file" value="$(find ur_description)/config/${ur_type}/joint_limits.yaml" lazy_eval="false"/>
-    <xacro:property name="_kinematics_parameters_file" value="$(find ur_description)/config/${ur_type}/default_kinematics.yaml" lazy_eval="false"/>
-    <xacro:property name="_physical_parameters_file" value="$(find ur_description)/config/${ur_type}/physical_parameters.yaml" lazy_eval="false"/>
-    <xacro:property name="_visual_parameters_file" value="$(find ur_description)/config/${ur_type}/visual_parameters.yaml" lazy_eval="false"/>
+    <xacro:property name="_joint_limits_parameters_file" value="$(find rc_manipulators_description)/urdf/arm/ur_description_webots/config/${ur_type}/joint_limits.yaml" lazy_eval="false"/>
+    <xacro:property name="_kinematics_parameters_file" value="$(find rc_manipulators_description)/urdf/arm/ur_description_webots/config/${ur_type}/default_kinematics.yaml" lazy_eval="false"/>
+    <xacro:property name="_physical_parameters_file" value="$(find rc_manipulators_description)/urdf/arm/ur_description_webots/config/${ur_type}/physical_parameters.yaml" lazy_eval="false"/>
+    <xacro:property name="_visual_parameters_file" value="$(find rc_manipulators_description)/urdf/arm/ur_description_webots/config/${ur_type}/visual_parameters.yaml" lazy_eval="false"/>
     <xacro:property name="_safety_limits" value="false" lazy_eval="false"/>
     <xacro:property name="_safety_pos_margin" value="0.15" lazy_eval="false"/>
@@ -208,7 +208,5 @@
     <!-- Universal Robots ROS2 Description -->
     <xacro:ur_robot
-      name="${name}"
-      tf_prefix="${_tf_prefix}"
-      parent="${parent_link}"
+      prefix="${_tf_prefix}"
       joint_limits_parameters_file="${_joint_limits_parameters_file}"
       kinematics_parameters_file="${_kinematics_parameters_file}"
@@ -217,50 +215,12 @@
       safety_limits="${_safety_limits}"
       safety_pos_margin="${_safety_pos_margin}"
-      safety_k_position="${_safety_k_position}">
-      <xacro:insert_block name="origin"/>
-    </xacro:ur_robot>
+      safety_k_position="${_safety_k_position}" />
+    <!-- Attach the arm to the parent link -->
+    <joint name="${_tf_prefix}base_joint" type="fixed">
+      <parent link="${parent_link}" />
+      <child link="${_tf_prefix}base_link" />
+      <xacro:insert_block name="origin" />
+    </joint>
     <!-- Use the right ros2_control depending on sim vs real -->
-    <xacro:if value="${_sim_ignition}">
-      <ros2_control name="${name}_hardware" type="system">
-        <hardware>
-          <!-- <plugin>gz_ros2_control/GazeboSimSystem</plugin> -->
-          <plugin>webots_ros2_control::Ros2ControlSystem</plugin>
-        </hardware>
-        <joint name="${name}_shoulder_pan_joint">
-          <command_interface name="position"/>
-          <state_interface name="position"/>
-          <state_interface name="velocity"/>
-        </joint>
-        <joint name="${name}_shoulder_lift_joint">
-          <command_interface name="position"/>
-          <state_interface name="position"/>
-          <state_interface name="velocity"/>
-        </joint>
-        <joint name="${name}_elbow_joint">
-          <command_interface name="position"/>
-          <state_interface name="position"/>
-          <state_interface name="velocity"/>
-        </joint>
-        <joint name="${name}_wrist_1_joint">
-          <command_interface name="position"/>
-          <state_interface name="position"/>
-          <state_interface name="velocity"/>
-        </joint>
-        <joint name="${name}_wrist_2_joint">
-          <command_interface name="position"/>
-          <state_interface name="position"/>
-          <state_interface name="velocity"/>
-        </joint>
-        <joint name="${name}_wrist_3_joint">
-          <command_interface name="position"/>
-          <state_interface name="position"/>
-          <state_interface name="velocity"/>
-        </joint>
-      </ros2_control>
-      <!-- <gazebo> -->
-        <!-- <plugin filename="gz_ros2_control-system" -->
-                <!-- name="gz_ros2_control::GazeboSimROS2ControlPlugin"/> -->
-      <!-- </gazebo> -->
-    </xacro:if>
     <!-- REAL ROBOT: only include the UR driver when NOT sim -->
     <xacro:unless value="${_sim_ignition}">

File: rc_platform_description/urdf/a300/a300.urdf.xacro (robot description, xacro)
@@ -33,5 +33,11 @@
     <xacro:property name="top_z" value="${chassis_z_size}"/>
     <!-- Base Link: center of rotation at the bottom of the robot -->
-    <link name="base_link"/>
+    <link name="base_link">
+      <inertial>
+        <mass value="0.1"/>
+        <origin xyz="0 0 0" rpy="0 0 0"/>
+        <inertia ixx="0.001" ixy="0" ixz="0" iyy="0.001" iyz="0" izz="0.001"/>
+      </inertial>
+    </link>
     <!-- Chassis Link: center of the bottom of the robot chassis -->
     <link name="chassis_link">

File: rc_platform_description/urdf/a300/drivetrain/motor.urdf.xacro (robot description, xacro)
@@ -3,5 +3,4 @@
   <xacro:macro name="a300_motor" params="prefix side">
     <xacro:property name="rotation_yaw" value="${math.pi if side == 'left' else 0}"/>
-    <xacro:property name="translation_y" value="${0.0655 if side == 'left' else -0.0655}"/>
     <link name="${prefix}_${side}_motor_link">
       <visual>
@@ -23,10 +22,4 @@
       <origin rpy="0 0 0"/>
     </joint>
-    <link name="${prefix}_${side}_motor_mount"/>
-    <joint name="${prefix}_${side}_motor_mount_joint" type="fixed">
-      <parent link="${prefix}_${side}_motor_link"/>
-      <child link="${prefix}_${side}_motor_mount"/>
-      <origin xyz="0 ${translation_y} 0"/>
-    </joint>
   </xacro:macro>
 </robot>

File: rc_platform_description/urdf/a300/drivetrain/wheels/outdoor.urdf.xacro (robot description, xacro)
@@ -5,4 +5,5 @@
   <xacro:property name="a300_outdoor_wheel_width" value="0.1143" />
   <xacro:macro name="a300_outdoor_wheel" params="prefix side">
+    <xacro:property name="translation_y" value="${0.0655 if side == 'left' else -0.0655}"/>
     <link name="${prefix}_${side}_wheel_link">
       <inertial>
@@ -39,5 +40,6 @@
     <!-- </gazebo> -->
     <joint name="${prefix}_${side}_wheel_joint" type="continuous">
-      <parent link="${prefix}_${side}_motor_mount"/>
+      <origin xyz="0 ${translation_y} 0" rpy="0 0 0"/>
+      <parent link="${prefix}_${side}_motor_link"/>
       <child link="${prefix}_${side}_wheel_link"/>
       <axis xyz="0 1 0" rpy="0 0 0" />

File: rc_platform_description/urdf/generic/gazebo.urdf.xacro (robot description, xacro)
@@ -2,5 +2,5 @@
 <robot xmlns:xacro="http://ros.org/wiki/xacro">
   <xacro:if value="$(arg is_sim)">
-    <ros2_control name="WebotsControl" type="system">
+    <ros2_control name="WebotsPlatformControl" type="system">
       <hardware>
         <plugin>webots_ros2_control::Ros2ControlSystem</plugin>

File: rc_sensors_description/urdf/hokuyo_ust.urdf.xacro (robot description, xacro)
@@ -13,4 +13,15 @@
         <material name="rc_dark_grey" />
       </visual>
+      <collision>
+        <origin xyz="0 0 0" rpy="0 0 0" />
+        <geometry>
+          <mesh filename="package://rc_sensors_description/meshes/hokuyo_ust.stl" />
+        </geometry>
+      </collision>
+      <inertial>
+        <mass value="0.1" />
+        <origin xyz="0 0 0" />
+        <inertia ixx="0.0001" ixy="0.0" ixz="0.0" iyy="0.0001" iyz="0.0" izz="0.0001" />
+      </inertial>
     </link>
     <link name="${name}_laser">
@@ -35,34 +46,80 @@
     </joint>
     <xacro:property name="samples" value="${round((max_ang - min_ang) * 180 / (ang_res * pi))}"/>
-    <gazebo reference="${name}_laser">
-      <sensor name="${name}" type="gpu_lidar">
-        <update_rate>${update_rate}</update_rate>
-        <visualize>true</visualize>
-        <always_on>true</always_on>
-        <gz_frame_id>${name}_laser</gz_frame_id>
-        <topic>$(arg namespace)/sensors/${name}/scan</topic>
-        <lidar>
-          <scan>
-            <horizontal>
-              <samples>${samples}</samples>
-              <resolution>1</resolution>
-              <min_angle>${min_ang}</min_angle>
-              <max_angle>${max_ang}</max_angle>
-            </horizontal>
-            <vertical>
-              <samples>1</samples>
-              <resolution>1</resolution>
-              <min_angle>0</min_angle>
-              <max_angle>0</max_angle>
-            </vertical>
-          </scan>
-          <range>
-            <min>${min_range}</min>
-            <max>${max_range}</max>
-            <resolution>0.01</resolution>
-          </range>
-        </lidar>
-      </sensor>
-    </gazebo>
+    <xacro:arg name="is_sim" default="false" />
+    <xacro:if value="$(arg is_sim)">
+      <gazebo reference="${name}_laser">
+        <sensor name="${name}" type="ray">
+          <update_rate>${update_rate}</update_rate>
+          <visualize>true</visualize>
+          <always_on>true</always_on>
+          <gz_frame_id>${name}_laser</gz_frame_id>
+          <topic>$(arg namespace)/sensors/${name}/scan</topic>
+          <lidar>
+            <scan>
+              <horizontal>
+                <samples>${samples}</samples>
+                <resolution>1</resolution>
+                <min_angle>${min_ang}</min_angle>
+                <max_angle>${max_ang}</max_angle>
+              </horizontal>
+              <vertical>
+                <samples>1</samples>
+                <resolution>1</resolution>
+                <min_angle>0</min_angle>
+                <max_angle>0</max_angle>
+              </vertical>
+            </scan>
+            <range>
+              <min>${min_range}</min>
+              <max>${max_range}</max>
+              <resolution>0.01</resolution>
+            </range>
+          </lidar>
+        </sensor>
+      </gazebo>
+      <webots>
+        <device reference="${name}" type="Lidar">
+          <ros>
+            <enabled>true</enabled>
+            <updateRate>${update_rate}</updateRate>
+            <topicName>$(arg namespace)/sensors/${name}/scan</topicName>
+            <alwaysOn>true</alwaysOn>
+            <frameName>${name}_laser</frameName>
+          </ros>
+        </device>
+      </webots>
+    </xacro:if>
+    <xacro:unless value="$(arg is_sim)">
+      <gazebo reference="${name}_laser">
+        <sensor name="${name}" type="gpu_lidar">
+          <update_rate>${update_rate}</update_rate>
+          <visualize>true</visualize>
+          <always_on>true</always_on>
+          <gz_frame_id>${name}_laser</gz_frame_id>
+          <topic>$(arg namespace)/sensors/${name}/scan</topic>
+          <lidar>
+            <scan>
+              <horizontal>
+                <samples>${samples}</samples>
+                <resolution>1</resolution>
+                <min_angle>${min_ang}</min_angle>
+                <max_angle>${max_ang}</max_angle>
+              </horizontal>
+              <vertical>
+                <samples>1</samples>
+                <resolution>1</resolution>
+                <min_angle>0</min_angle>
+                <max_angle>0</max_angle>
+              </vertical>
+            </scan>
+            <range>
+              <min>${min_range}</min>
+              <max>${max_range}</max>
+              <resolution>0.01</resolution>
+            </range>
+          </lidar>
+        </sensor>
+      </gazebo>
+    </xacro:unless>
   </xacro:macro>
 </robot>

File: rc_sensors_description/urdf/intel_realsense.urdf.xacro (robot description, xacro)
@@ -33,26 +33,59 @@
       </xacro:sensor_d456>
     </xacro:if>
-    <gazebo reference="${name}_link">
-      <sensor name="${name}" type="rgbd_camera">
-        <camera>
-          <horizontal_fov>1.25</horizontal_fov>
-          <image>
-            <width>${image_width}</width>
-            <height>${image_height}</height>
-          </image>
-          <clip>
-            <near>0.3</near>
-            <far>100</far>
-          </clip>
+    <xacro:arg name="is_sim" default="false" />
+    <xacro:if value="$(arg is_sim)">
+      <gazebo reference="${name}_link">
+        <sensor name="${name}" type="camera">
+          <camera>
+            <horizontal_fov>1.25</horizontal_fov>
+            <image>
+              <width>${image_width}</width>
+              <height>${image_height}</height>
+            </image>
+            <clip>
+              <near>0.3</near>
+              <far>100</far>
+            </clip>
+          </camera>
+          <always_on>1</always_on>
+          <update_rate>${update_rate}</update_rate>
+        </sensor>
+      </gazebo>
+      <webots>
+        <device reference="${name}" type="Camera">
+          <ros>
+            <enabled>true</enabled>
+            <updateRate>${update_rate}</updateRate>
+            <topicName>$(arg namespace)/sensors/${name}</topicName>
+            <alwaysOn>true</alwaysOn>
+            <frameName>${name}_link</frameName>
+          </ros>
+        </device>
+      </webots>
+    </xacro:if>
+    <xacro:unless value="$(arg is_sim)">
+      <gazebo reference="${name}_link">
+        <sensor name="${name}" type="rgbd_camera">
+          <camera>
+            <horizontal_fov>1.25</horizontal_fov>
+            <image>
+              <width>${image_width}</width>
+              <height>${image_height}</height>
+            </image>
+            <clip>
+              <near>0.3</near>
+              <far>100</far>
+            </clip>
+            <gz_frame_id>${name}_link</gz_frame_id>
+            <optical_frame_id>${name}_color_optical_frame</optical_frame_id>
+          </camera>
+          <always_on>1</always_on>
+          <update_rate>${update_rate}</update_rate>
+          <visualize>true</visualize>
           <gz_frame_id>${name}_link</gz_frame_id>
-          <optical_frame_id>${name}_color_optical_frame</optical_frame_id>
-        </camera>
-        <always_on>1</always_on>
-        <update_rate>${update_rate}</update_rate>
-        <visualize>true</visualize>
-        <gz_frame_id>${name}_link</gz_frame_id>
-        <topic>$(arg namespace)/sensors/${name}</topic>
-      </sensor>
-    </gazebo>
+          <topic>$(arg namespace)/sensors/${name}</topic>
+        </sensor>
+      </gazebo>
+    </xacro:unless>
   </xacro:macro>
 </robot>

File: rc_sensors_description/urdf/microstrain_imu.urdf.xacro (robot description, xacro)
@@ -10,4 +10,9 @@
         <material name="rc_dark_grey" />
       </visual>
+      <inertial>
+        <mass value="0.1"/>
+        <origin xyz="0 0 0" rpy="0 0 0"/>
+        <inertia ixx="0.001" ixy="0" ixz="0" iyy="0.001" iyz="0" izz="0.001"/>
+      </inertial>
     </link>
     <joint name="${name}_base_joint" type="fixed">
@@ -21,13 +26,35 @@
       <child link="${name}_link" />
     </joint>
-    <gazebo reference="${name}_link">
-      <sensor type="imu" name="${name}">
-        <always_on>true</always_on>
-        <update_rate>${update_rate}</update_rate>
-        <visualize>true</visualize>
-        <gz_frame_id>${name}_link</gz_frame_id>
-        <topic>$(arg namespace)/sensors/${name}/data</topic>
-      </sensor>
-    </gazebo>
+    <xacro:arg name="is_sim" default="false" />
+    <xacro:if value="$(arg is_sim)">
+      <gazebo reference="${name}_link">
+        <plugin filename="libgazebo_ros_imu_sensor.so" name="${name}_imu_plugin">
+          <topicName>${name}</topicName>
+        </plugin>
+      </gazebo>
+      <webots>
+        <plugin type="webots_ros2_driver::Ros2IMU">
+          <enabled>true</enabled>
+          <updateRate>${update_rate}</updateRate>
+          <topicName>$(arg namespace)/sensors/${name}/data</topicName>
+          <alwaysOn>true</alwaysOn>
+          <frameName>${name}_link</frameName>
+          <inertialUnitName>${name} inertial</inertialUnitName>
+          <gyroName>${name} gyro</gyroName>
+          <accelerometerName>${name} accelerometer</accelerometerName>
+        </plugin>
+      </webots>
+    </xacro:if>
+    <xacro:unless value="$(arg is_sim)">
+      <gazebo reference="${name}_link">
+        <sensor type="imu" name="${name}">
+          <always_on>true</always_on>
+          <update_rate>${update_rate}</update_rate>
+          <visualize>true</visualize>
+          <gz_frame_id>${name}_link</gz_frame_id>
+          <topic>$(arg namespace)/sensors/${name}/data</topic>
+        </sensor>
+      </gazebo>
+    </xacro:unless>
   </xacro:macro>
 </robot>
