Commit message: Webots port finished: + Tested moveit + Tested Mapping using slam toolbox + Tested navigation using Nav2

File: rc_common/robot.urdf.xacro (robot description, xacro)
@@ -37,4 +37,8 @@
     <origin xyz="0.445 0.0 0.1" rpy="0.0 0.0 0.0"/>
   </xacro:intel_realsense>
+  <!-- camera_1 -->
+  <xacro:intel_realsense name="camera_1" parent_link="arm_0_wrist_3_link" update_rate="30" image_height="480" image_width="640" model="d435">
+    <origin xyz="0.0 -0.05 -0.05" rpy="-2.362919 -1.570368 -2.362919"/>
+  </xacro:intel_realsense>
   <!-- imu_0 -->
   <xacro:include filename="$(find rc_sensors_description)/urdf/microstrain_imu.urdf.xacro"/>

File: rc_sensors_description/urdf/hokuyo_ust.urdf.xacro (robot description, xacro)
@@ -41,5 +41,5 @@
     <joint name="${name}_laser_joint" type="fixed">
       <!-- This offset is from the base of the bracket to the LIDAR's focal point. -->
-      <origin xyz="0 0 0.0474" rpy="0 0 0" />
+      <origin xyz="0 0 0.0474" rpy="3.141592653589793 0 0" />
       <parent link="${name}_link" />
       <child link="${name}_laser" />
@@ -55,5 +55,5 @@
           <gz_frame_id>${name}_laser</gz_frame_id>
           <topic>$(arg namespace)/sensors/${name}/scan</topic>
-          <lidar>
+          <ray>
             <scan>
               <horizontal>
@@ -75,5 +75,5 @@
               <resolution>0.01</resolution>
             </range>
-          </lidar>
+          </ray>
         </sensor>
       </gazebo>

File: rc_sensors_description/urdf/intel_realsense.urdf.xacro (robot description, xacro)
@@ -11,5 +11,5 @@
     <xacro:if value="${model == 'd435'}">
       <xacro:include filename="$(find rc_sensors_description)/urdf/intel/d435.urdf.xacro" />
-      <xacro:sensor_d435 name="${name}" parent="${parent_link}">
+      <xacro:sensor_d435 name="${name}" parent="${parent_link}" use_nominal_extrinsics="true">
         <xacro:insert_block name="origin" />
       </xacro:sensor_d435>
@@ -35,5 +35,5 @@
     <xacro:arg name="is_sim" default="false" />
     <xacro:if value="$(arg is_sim)">
-      <gazebo reference="${name}_link">
+      <gazebo reference="${name}_color_optical_frame">
         <sensor name="${name}" type="camera">
           <camera>
@@ -52,4 +52,21 @@
         </sensor>
       </gazebo>
+      <gazebo reference="${name}_color_optical_frame">
+        <sensor name="${name}_depth" type="depth">
+          <camera>
+            <horizontal_fov>1.25</horizontal_fov>
+            <image>
+              <width>${image_width}</width>
+              <height>${image_height}</height>
+            </image>
+            <clip>
+              <near>0.1</near>
+              <far>200</far>
+            </clip>
+          </camera>
+          <always_on>1</always_on>
+          <update_rate>${update_rate}</update_rate>
+        </sensor>
+      </gazebo>
       <webots>
         <device reference="${name}" type="Camera">
@@ -59,6 +76,19 @@
             <topicName>$(arg namespace)/sensors/${name}</topicName>
             <alwaysOn>true</alwaysOn>
-            <frameName>${name}_link</frameName>
+            <frameName>${name}_color_optical_frame</frameName>
           </ros>
+        </device>
+        <device reference="${name}_depth" type="RangeFinder">
+          <ros>
+            <enabled>true</enabled>
+            <updateRate>${update_rate}</updateRate>
+            <topicName>$(arg namespace)/sensors/${name}/depth</topicName>
+            <imageSuffix>/image_raw</imageSuffix>
+            <pointCloudSuffix>/points</pointCloudSuffix>
+            <alwaysOn>true</alwaysOn>
+            <frameName>${name}_color_optical_frame</frameName>
+          </ros>
+          <minRange>0.1</minRange>
+          <maxRange>20.0</maxRange>
         </device>
       </webots>
